File: PCB/arduino-encoder.sch (KiCad schematic (older format))
At the start: 0 parts

Commit message: add ws2812 circuit,
Parts:
- added H1, H2, H3, H4: MOUNT_M3, MountingHole:MountingHole_3.2mm_M3, symbol taobao-mounting-hole:MOUNT_M3
Changed lines of the file:
@@
 $Descr A4 11693 8268
 encoding utf-8
-Sheet 1 1
+Sheet 1 2
 Title ""
 Date ""
@@
 Data
 89 50 4E 47 0D 0A 1A 0A 00 00 00 0D 49 48 44 52 00 00 04 00 00 00 01 EA 08 02 00 00 00 15 98 AB
-97 00 00 00 03 73 42 49 54 08 08 08 DB E1 4F E0 00 00 00 09 70 48 59 73 00 00 0B 12 00 00 0B 12
-01 D2 DD 7E FC 00 00 20 00 49 44 41 54 78 9C EC DD D9 8F 25 59 7A 18 F6 EF EC B1 DF 3D 97 CA AC
+97 00 00 00 03 73 42 49 54 08 08 08 DB E1 4F E0 00 00 00 09 70 48 59 73 00 00 0A F0 00 00 0A F0
+01 42 AC 34 98 00 00 20 00 49 44 41 54 78 9C EC DD D9 8F 25 59 7A 18 F6 EF EC B1 DF 3D 97 CA AC
 EC EA EA EA 9E E1 6C F2 90 22 45 52 A4 48 C8 F0 22 03 06 6C C0 EF 7E F1 8B FF 0B FE 45 82 01 C3
 12 40 89 02 4C 88 22 39 5C 86 C3 E1 CC F4 56 6B 56 EE 77 8F F5 AC 9F 1F 6E 55 76 4D 57 15 67 9A
@@
 EndData
 $EndBitmap
+$Comp
+L taobao-mounting-hole:MOUNT_M3 H1
+U 1 1 5E10C653
+P 5950 6550
+F 0 "H1" H 6050 6596 50  0000 L CNN
+F 1 "MOUNT_M3" H 6050 6505 50  0000 L CNN
+F 2 "MountingHole:MountingHole_3.2mm_M3" H 5950 6550 50  0001 C CNN
+F 3 "~" H 5950 6550 50  0001 C CNN
+	1    5950 6550
+	1    0    0    -1
+$EndComp
+$Comp
+L taobao-mounting-hole:MOUNT_M3 H2
+U 1 1 5E10C7C5
+P 5950 6800
+F 0 "H2" H 6050 6846 50  0000 L CNN
+F 1 "MOUNT_M3" H 6050 6755 50  0000 L CNN
+F 2 "MountingHole:MountingHole_3.2mm_M3" H 5950 6800 50  0001 C CNN
+F 3 "~" H 5950 6800 50  0001 C CNN
+	1    5950 6800
+	1    0    0    -1
+$EndComp
+$Comp
+L taobao-mounting-hole:MOUNT_M3 H3
+U 1 1 5E10CAB5
+P 5950 7000
+F 0 "H3" H 6050 7046 50  0000 L CNN
+F 1 "MOUNT_M3" H 6050 6955 50  0000 L CNN
+F 2 "MountingHole:MountingHole_3.2mm_M3" H 5950 7000 50  0001 C CNN
+F 3 "~" H 5950 7000 50  0001 C CNN
+	1    5950 7000
+	1    0    0    -1
+$EndComp
+$Comp
+L taobao-mounting-hole:MOUNT_M3 H4
+U 1 1 5E10CC9D
+P 5950 7200
+F 0 "H4" H 6050 7246 50  0000 L CNN
+F 1 "MOUNT_M3" H 6050 7155 50  0000 L CNN
+F 2 "MountingHole:MountingHole_3.2mm_M3" H 5950 7200 50  0001 C CNN
+F 3 "~" H 5950 7200 50  0001 C CNN
+	1    5950 7200
+	1    0    0    -1
+$EndComp
+$Sheet
+S 7700 4350 700  650
+U 5E117B87
+F0 "ws2812.sch" 50
+F1 "ws2812.sch" 50
+$EndSheet
 $EndSCHEMATC
